File: hardware/Class D Amplifier - TPA3122/TPA3122_Class-D.sch (EAGLE design)
At the start: 49 parts, among them CN1 Left_Speaker, CN2 Right_Speaker, CN3 Power_Supply, J1 SJ-3523-SMT, J4 POWER_JACKSLT, Q1 FQP47P06, U1 TPA3122D2_N_20

Commit message: Fixed GND mistake in Barrel Jack
Connections:
- net GND: now also J4.GNDBREAK
Changed lines of the file:
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@@
 <wire x1="15.24" y1="127" x2="20.32" y2="127" width="0.1524" layer="91"/>
 <wire x1="20.32" y1="127" x2="20.32" y2="124.46" width="0.1524" layer="91"/>
+<pinref part="J4" gate="G$1" pin="GNDBREAK"/>
+<wire x1="15.24" y1="129.54" x2="20.32" y2="129.54" width="0.1524" layer="91"/>
+<wire x1="20.32" y1="129.54" x2="20.32" y2="127" width="0.1524" layer="91"/>
+<junction x="20.32" y="127"/>
 </segment>
 </net>
