File: hardware/TPA3122/TPA3122_Class-D.brd (EAGLE design)
At the start: 70 x 56.4 mm, 49 parts, among them CN1 Left_Speaker, CN2 Right_Speaker, CN3 Power_Supply, J1 SJ-3523-SMT, J4 POWER_JACKSLT, Q1 FQP47P06, U1 TPA3122D2_N_20

Commit message: Corrected TPA3122 Power Jack
Parts:
- J4: device SparkFun-Connectors:POWER_JACK_SLOT -> TPA3122:POWER_JACK_SLOT
- moved J4 1.27 mm to (55.2, 72.4)
Routing:
- net EXT-POWER: track 14.3 -> 16.0 mm
Changed lines of the file:
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@@
 <?xml version="1.0" encoding="utf-8"?>
 <!DOCTYPE eagle SYSTEM "eagle.dtd">
-<eagle version="8.4.0">
+<eagle version="8.7.1">
 <drawing>
 <settings>
@@
 <layer number="20" name="Dimension" color="24" fill="1" visible="yes" active="yes"/>
 <layer number="21" name="tPlace" color="7" fill="1" visible="yes" active="yes"/>
-<layer number="22" name="bPlace" color="7" fill="1" visible="yes" active="yes"/>
+<layer number="22" name="bPlace" color="7" fill="1" visible="no" active="yes"/>
 <layer number="23" name="tOrigins" color="15" fill="1" visible="yes" active="yes"/>
 <layer number="24" name="bOrigins" color="15" fill="1" visible="no" active="yes"/>
@@
 <layer number="38" name="bTest" color="7" fill="1" visible="no" active="yes"/>
 <layer number="39" name="tKeepout" color="4" fill="11" visible="yes" active="yes"/>
-<layer number="40" name="bKeepout" color="1" fill="11" visible="yes" active="yes"/>
+<layer number="40" name="bKeepout" color="1" fill="11" visible="no" active="yes"/>
 <layer number="41" name="tRestrict" color="4" fill="10" visible="yes" active="yes"/>
-<layer number="42" name="bRestrict" color="1" fill="10" visible="yes" active="yes"/>
+<layer number="42" name="bRestrict" color="1" fill="10" visible="no" active="yes"/>
 <layer number="43" name="vRestrict" color="2" fill="10" visible="no" active="yes"/>
 <layer number="44" name="Drills" color="7" fill="1" visible="no" active="yes"/>
 <layer number="45" name="Holes" color="7" fill="1" visible="yes" active="yes"/>
-<layer number="46" name="Milling" color="41" fill="1" visible="no" active="yes"/>
+<layer number="46" name="Milling" color="41" fill="1" visible="yes" active="yes"/>
 <layer number="47" name="Measures" color="7" fill="1" visible="no" active="yes"/>
 <layer number="48" name="Document" color="7" fill="1" visible="no" active="yes"/>
@@
 <param name="dpMaxLengthDifference" value="10mm"/>
 <param name="dpGapFactor" value="2.5"/>
+<param name="checkAngle" value="0"/>
 <param name="checkFont" value="1"/>
 <param name="checkRestrict" value="1"/>
 <param name="checkStop" value="0"/>
+<param name="checkValues" value="0"/>
 <param name="useDiameter" value="13"/>
 <param name="maxErrors" value="50"/>
@@
 <attribute name="VALUE" x="55.245" y="19.939" size="0.0254" layer="27"/>
 </element>
-<element name="J4" library="SparkFun-Connectors" package="POWER_JACK_SLOT" value="POWER_JACKSLT" x="56.515" y="72.39" smashed="yes" rot="R180">
-<attribute name="NAME" x="45.085" y="66.675" size="1.778" layer="25" rot="R270"/>
-<attribute name="VALUE" x="45.085" y="72.39" size="1.778" layer="27" rot="R270"/>
+<element name="J4" library="TPA3122" package="POWER_JACK_SLOT" value="POWER_JACKSLT" x="55.245" y="72.39" smashed="yes" rot="R180">
+<attribute name="NAME" x="43.815" y="66.675" size="1.778" layer="25" rot="R270"/>
+<attribute name="VALUE" x="43.815" y="72.39" size="1.778" layer="27" rot="R270"/>
 </element>
 <element name="J3" library="SparkFun-Connectors" library_urn="urn:adsk.eagle:library:513" package="1X01" package3d_urn="urn:adsk.eagle:package:38028/1" value="" x="16.51" y="26.797" smashed="yes">
@@
 <contactref element="J4" pad="PWR"/>
 <wire x1="50.165" y1="55.245" x2="53.51" y2="58.59" width="1.016" layer="1" curve="-90"/>
-<wire x1="53.935" y1="58.59" x2="53.51" y2="58.59" width="0.6096" layer="1"/>
+<wire x1="52.665" y1="58.59" x2="53.51" y2="58.59" width="0.6096" layer="1"/>
 <wire x1="61.295" y1="62.935" x2="56.95" y2="58.59" width="1.016" layer="1" curve="-90"/>
-<wire x1="56.95" y1="58.59" x2="53.935" y2="58.59" width="1.016" layer="1"/>
+<wire x1="56.95" y1="58.59" x2="52.665" y2="58.59" width="1.016" layer="1"/>
 </signal>
 <signal name="RIGHT">
